Commit message: Set positive mobile joint limits for Lula

File: humanoid_urdf_assemble/urdf/combined_mobile_humanoid_base.urdf (robot description, URDF)
Before this commit: robot combined_mobile_humanoid, 24 links, 23 joints
Joints:
- joint joint1_mobile: limit lower=0 upper=0 effort=0 velocity=0 -> lower=0 upper=0 effort=1.0 velocity=1.0
- joint joint2_mobile: limit lower=0 upper=0 effort=0 velocity=0 -> lower=0 upper=0 effort=1.0 velocity=1.0
- joint joint3_mobile: limit lower=0 upper=0 effort=0 velocity=0 -> lower=0 upper=0 effort=1.0 velocity=1.0
- joint joint4_mobile: limit lower=0 upper=0 effort=0 velocity=0 -> lower=0 upper=0 effort=1.0 velocity=1.0
- joint joint5_mobile: limit lower=0 upper=0 effort=0 velocity=0 -> lower=0 upper=0 effort=1.0 velocity=1.0
- joint joint6_mobile: limit lower=0 upper=0 effort=0 velocity=0 -> lower=0 upper=0 effort=1.0 velocity=1.0
- joint joint7_mobile: limit lower=0 upper=0 effort=0 velocity=0 -> lower=0 upper=0 effort=1.0 velocity=1.0
- joint joint8_mobile: limit lower=0 upper=0 effort=0 velocity=0 -> lower=0 upper=0 effort=1.0 velocity=1.0

File: humanoid_urdf_assemble/urdf/combined_mobile_v4_onlyarm.urdf (robot description, URDF)
Before this commit: robot combined_mobile_v4_onlyarm, 26 links, 25 joints
Joints:
- joint joint1_mobile: limit lower=0 upper=0 effort=0 velocity=0 -> lower=0 upper=0 effort=1.0 velocity=1.0
- joint joint2_mobile: limit lower=0 upper=0 effort=0 velocity=0 -> lower=0 upper=0 effort=1.0 velocity=1.0
- joint joint3_mobile: limit lower=0 upper=0 effort=0 velocity=0 -> lower=0 upper=0 effort=1.0 velocity=1.0
- joint joint4_mobile: limit lower=0 upper=0 effort=0 velocity=0 -> lower=0 upper=0 effort=1.0 velocity=1.0
- joint joint5_mobile: limit lower=0 upper=0 effort=0 velocity=0 -> lower=0 upper=0 effort=1.0 velocity=1.0
- joint joint6_mobile: limit lower=0 upper=0 effort=0 velocity=0 -> lower=0 upper=0 effort=1.0 velocity=1.0
- joint joint7_mobile: limit lower=0 upper=0 effort=0 velocity=0 -> lower=0 upper=0 effort=1.0 velocity=1.0
- joint joint8_mobile: limit lower=0 upper=0 effort=0 velocity=0 -> lower=0 upper=0 effort=1.0 velocity=1.0

Commit message: Relax mobile joint limits and force

File: humanoid_urdf_assemble/urdf/combined_mobile_humanoid_base.urdf (robot description, URDF)
Before this commit: robot combined_mobile_humanoid, 24 links, 23 joints
Joints:
- joint joint1_mobile: limit lower=0 upper=0 effort=0 velocity=0 -> lower=-3.14159 upper=3.14159 effort=500.0 velocity=2.0
- joint joint2_mobile: limit lower=0 upper=0 effort=0 velocity=0 -> lower=-3.14159 upper=3.14159 effort=500.0 velocity=2.0
- joint joint3_mobile: limit lower=0 upper=0 effort=0 velocity=0 -> lower=-3.14159 upper=3.14159 effort=500.0 velocity=2.0
- joint joint4_mobile: limit lower=0 upper=0 effort=0 velocity=0 -> lower=-3.14159 upper=3.14159 effort=500.0 velocity=2.0
- joint joint5_mobile: limit lower=0 upper=0 effort=0 velocity=0 -> lower=-3.14159 upper=3.14159 effort=500.0 velocity=2.0
- joint joint6_mobile: limit lower=0 upper=0 effort=0 velocity=0 -> lower=-3.14159 upper=3.14159 effort=500.0 velocity=2.0
- joint joint7_mobile: limit lower=0 upper=0 effort=0 velocity=0 -> lower=-3.14159 upper=3.14159 effort=500.0 velocity=2.0
- joint joint8_mobile: limit lower=0 upper=0 effort=0 velocity=0 -> lower=-3.14159 upper=3.14159 effort=500.0 velocity=2.0

File: humanoid_urdf_assemble/urdf/combined_mobile_v4_onlyarm.urdf (robot description, URDF)
Before this commit: robot combined_mobile_v4_onlyarm, 26 links, 25 joints
Joints:
- joint joint1_mobile: limit lower=0 upper=0 effort=0 velocity=0 -> lower=-3.14159 upper=3.14159 effort=500.0 velocity=2.0
- joint joint2_mobile: limit lower=0 upper=0 effort=0 velocity=0 -> lower=-3.14159 upper=3.14159 effort=500.0 velocity=2.0
- joint joint3_mobile: limit lower=0 upper=0 effort=0 velocity=0 -> lower=-3.14159 upper=3.14159 effort=500.0 velocity=2.0
- joint joint4_mobile: limit lower=0 upper=0 effort=0 velocity=0 -> lower=-3.14159 upper=3.14159 effort=500.0 velocity=2.0
- joint joint5_mobile: limit lower=0 upper=0 effort=0 velocity=0 -> lower=-3.14159 upper=3.14159 effort=500.0 velocity=2.0
- joint joint6_mobile: limit lower=0 upper=0 effort=0 velocity=0 -> lower=-3.14159 upper=3.14159 effort=500.0 velocity=2.0
- joint joint7_mobile: limit lower=0 upper=0 effort=0 velocity=0 -> lower=-3.14159 upper=3.14159 effort=500.0 velocity=2.0
- joint joint8_mobile: limit lower=0 upper=0 effort=0 velocity=0 -> lower=-3.14159 upper=3.14159 effort=500.0 velocity=2.0

Commit message: Calibrate arm direction and mobile joints

File: humanoid_urdf_assemble/urdf/combined_mobile_humanoid_base.urdf (robot description, URDF)
Before this commit: robot combined_mobile_humanoid, 24 links, 23 joints
Joints:
- joint joint1_mobile: limit lower=0 upper=0 effort=0 velocity=0 -> lower=-3.14159 upper=3.14159 effort=5000.0 velocity=5.0
- joint joint2_mobile: limit lower=0 upper=0 effort=0 velocity=0 -> lower=-3.14159 upper=3.14159 effort=5000.0 velocity=5.0
- joint joint3_mobile: limit lower=0 upper=0 effort=0 velocity=0 -> lower=-3.14159 upper=3.14159 effort=5000.0 velocity=5.0
- joint joint4_mobile: limit lower=0 upper=0 effort=0 velocity=0 -> lower=-3.14159 upper=3.14159 effort=5000.0 velocity=5.0
- joint joint5_mobile: limit lower=0 upper=0 effort=0 velocity=0 -> lower=-3.14159 upper=3.14159 effort=5000.0 velocity=5.0
- joint joint6_mobile: limit lower=0 upper=0 effort=0 velocity=0 -> lower=-3.14159 upper=3.14159 effort=5000.0 velocity=5.0
- joint joint7_mobile: limit lower=0 upper=0 effort=0 velocity=0 -> lower=-3.14159 upper=3.14159 effort=5000.0 velocity=5.0
- joint joint8_mobile: limit lower=0 upper=0 effort=0 velocity=0 -> lower=-3.14159 upper=3.14159 effort=5000.0 velocity=5.0

File: humanoid_urdf_assemble/urdf/combined_mobile_v4_onlyarm.urdf (robot description, URDF)
Before this commit: robot combined_mobile_v4_onlyarm, 26 links, 25 joints
Joints:
- joint joint1_mobile: limit lower=0 upper=0 effort=0 velocity=0 -> lower=-3.14159 upper=3.14159 effort=5000.0 velocity=5.0
- joint joint2_mobile: limit lower=0 upper=0 effort=0 velocity=0 -> lower=-3.14159 upper=3.14159 effort=5000.0 velocity=5.0
- joint joint3_mobile: limit lower=0 upper=0 effort=0 velocity=0 -> lower=-3.14159 upper=3.14159 effort=5000.0 velocity=5.0
- joint joint4_mobile: limit lower=0 upper=0 effort=0 velocity=0 -> lower=-3.14159 upper=3.14159 effort=5000.0 velocity=5.0
- joint joint5_mobile: limit lower=0 upper=0 effort=0 velocity=0 -> lower=-3.14159 upper=3.14159 effort=5000.0 velocity=5.0
- joint joint6_mobile: limit lower=0 upper=0 effort=0 velocity=0 -> lower=-3.14159 upper=3.14159 effort=5000.0 velocity=5.0
- joint joint7_mobile: limit lower=0 upper=0 effort=0 velocity=0 -> lower=-3.14159 upper=3.14159 effort=5000.0 velocity=5.0
- joint joint8_mobile: limit lower=0 upper=0 effort=0 velocity=0 -> lower=-3.14159 upper=3.14159 effort=5000.0 velocity=5.0

Commit message: Prioritize z-axis mobile ladder joints

File: humanoid_urdf_assemble/urdf/combined_mobile_humanoid_base.urdf (robot description, URDF)
Before this commit: robot combined_mobile_humanoid, 24 links, 23 joints
Joints:
- joint joint1_mobile: limit lower=0 upper=0 effort=0 velocity=0 -> lower=-3.14159 upper=3.14159 effort=50000.0 velocity=5.0
- joint joint2_mobile: limit lower=0 upper=0 effort=0 velocity=0 -> lower=-3.14159 upper=3.14159 effort=50000.0 velocity=5.0
- joint joint3_mobile: limit lower=0 upper=0 effort=0 velocity=0 -> lower=-3.14159 upper=3.14159 effort=50000.0 velocity=5.0
- joint joint4_mobile: limit lower=0 upper=0 effort=0 velocity=0 -> lower=-3.14159 upper=3.14159 effort=50000.0 velocity=5.0
- joint joint5_mobile: limit lower=0 upper=0 effort=0 velocity=0 -> lower=-3.14159 upper=3.14159 effort=50000.0 velocity=5.0
- joint joint6_mobile: limit lower=0 upper=0 effort=0 velocity=0 -> lower=-3.14159 upper=3.14159 effort=50000.0 velocity=5.0
- joint joint7_mobile: limit lower=0 upper=0 effort=0 velocity=0 -> lower=-3.14159 upper=3.14159 effort=50000.0 velocity=5.0
- joint joint8_mobile: limit lower=0 upper=0 effort=0 velocity=0 -> lower=-3.14159 upper=3.14159 effort=50000.0 velocity=5.0

File: humanoid_urdf_assemble/urdf/combined_mobile_v4_onlyarm.urdf (robot description, URDF)
Before this commit: robot combined_mobile_v4_onlyarm, 26 links, 25 joints
Joints:
- joint joint1_mobile: limit lower=0 upper=0 effort=0 velocity=0 -> lower=-3.14159 upper=3.14159 effort=50000.0 velocity=5.0
- joint joint2_mobile: limit lower=0 upper=0 effort=0 velocity=0 -> lower=-3.14159 upper=3.14159 effort=50000.0 velocity=5.0
- joint joint3_mobile: limit lower=0 upper=0 effort=0 velocity=0 -> lower=-3.14159 upper=3.14159 effort=50000.0 velocity=5.0
- joint joint4_mobile: limit lower=0 upper=0 effort=0 velocity=0 -> lower=-3.14159 upper=3.14159 effort=50000.0 velocity=5.0
- joint joint5_mobile: limit lower=0 upper=0 effort=0 velocity=0 -> lower=-3.14159 upper=3.14159 effort=50000.0 velocity=5.0
- joint joint6_mobile: limit lower=0 upper=0 effort=0 velocity=0 -> lower=-3.14159 upper=3.14159 effort=50000.0 velocity=5.0
- joint joint7_mobile: limit lower=0 upper=0 effort=0 velocity=0 -> lower=-3.14159 upper=3.14159 effort=50000.0 velocity=5.0
- joint joint8_mobile: limit lower=0 upper=0 effort=0 velocity=0 -> lower=-3.14159 upper=3.14159 effort=50000.0 velocity=5.0

Commit message: Default mobile control to ladder lift joints

File: humanoid_urdf_assemble/urdf/combined_mobile_humanoid_base.urdf (robot description, URDF)
Before this commit: robot combined_mobile_humanoid, 24 links, 23 joints
Joints:
- joint joint1_mobile: limit lower=0 upper=0 effort=0 velocity=0 -> lower=-3.14159 upper=3.14159 effort=100000.0 velocity=5.0
- joint joint2_mobile: limit lower=0 upper=0 effort=0 velocity=0 -> lower=-3.14159 upper=3.14159 effort=100000.0 velocity=5.0
- joint joint3_mobile: limit lower=0 upper=0 effort=0 velocity=0 -> lower=-3.14159 upper=3.14159 effort=100000.0 velocity=5.0
- joint joint4_mobile: limit lower=0 upper=0 effort=0 velocity=0 -> lower=-3.14159 upper=3.14159 effort=100000.0 velocity=5.0
- joint joint5_mobile: limit lower=0 upper=0 effort=0 velocity=0 -> lower=-3.14159 upper=3.14159 effort=100000.0 velocity=5.0
- joint joint6_mobile: limit lower=0 upper=0 effort=0 velocity=0 -> lower=-3.14159 upper=3.14159 effort=100000.0 velocity=5.0
- joint joint7_mobile: limit lower=0 upper=0 effort=0 velocity=0 -> lower=-3.14159 upper=3.14159 effort=100000.0 velocity=5.0
- joint joint8_mobile: limit lower=0 upper=0 effort=0 velocity=0 -> lower=-3.14159 upper=3.14159 effort=100000.0 velocity=5.0

File: humanoid_urdf_assemble/urdf/combined_mobile_v4_onlyarm.urdf (robot description, URDF)
Before this commit: robot combined_mobile_v4_onlyarm, 26 links, 25 joints
Joints:
- joint joint1_mobile: limit lower=0 upper=0 effort=0 velocity=0 -> lower=-3.14159 upper=3.14159 effort=100000.0 velocity=5.0
- joint joint2_mobile: limit lower=0 upper=0 effort=0 velocity=0 -> lower=-3.14159 upper=3.14159 effort=100000.0 velocity=5.0
- joint joint3_mobile: limit lower=0 upper=0 effort=0 velocity=0 -> lower=-3.14159 upper=3.14159 effort=100000.0 velocity=5.0
- joint joint4_mobile: limit lower=0 upper=0 effort=0 velocity=0 -> lower=-3.14159 upper=3.14159 effort=100000.0 velocity=5.0
- joint joint5_mobile: limit lower=0 upper=0 effort=0 velocity=0 -> lower=-3.14159 upper=3.14159 effort=100000.0 velocity=5.0
- joint joint6_mobile: limit lower=0 upper=0 effort=0 velocity=0 -> lower=-3.14159 upper=3.14159 effort=100000.0 velocity=5.0
- joint joint7_mobile: limit lower=0 upper=0 effort=0 velocity=0 -> lower=-3.14159 upper=3.14159 effort=100000.0 velocity=5.0
- joint joint8_mobile: limit lower=0 upper=0 effort=0 velocity=0 -> lower=-3.14159 upper=3.14159 effort=100000.0 velocity=5.0
